File: TPS61165-heater-v2/TPS61165-heater-v2.kicad_pcb (KiCad board)
At the start: 2 copper layers, 44 x 35 mm, 20 parts, among them J1 USB_C_KoreanHroparts_6P, J2 A2001WV-2P, J3 Conn_01x02_Female, J4 A2001WV-2P, J5 MMCX, J6 Conn_01x02_Female, J7 MMCX, U1 TPS61165

Commit message: Update github
Parts:
- moved J7 17.9 mm to (141.8, 75.6)
- moved L1 12.3 mm to (151.3, 86.5), turned to 0 degrees
- moved JP1 10.9 mm to (143.8, 79.7)
- moved R2 9.52 mm to (141.2, 80.7), turned to 270 degrees
- moved R1 7.47 mm to (147.2, 76.5), turned to 90 degrees
- moved D1 6.04 mm to (154.9, 81.1)
- moved C1 5.13 mm to (150.4, 76.2), turned to 0 degrees
- moved R4 4.61 mm to (140.5, 70.7)
- moved R3 3.85 mm to (155.6, 75.2)
- moved C3 3.17 mm to (146.9, 80.2), turned to 90 degrees
- moved J5 2.30 mm to (134.3, 66.1)
- moved J4 2.30 mm to (151.8, 67.5), turned to 270 degrees
- moved J3 2.30 mm to (144.1, 67.5), turned to 0 degrees
- moved JP2 1.38 mm to (139.6, 68.0), turned to 270 degrees
- moved U1 1.34 mm to (150.2, 79.8), turned to 90 degrees
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Connections:
- U1 pad 1: Net-(J3-Pad2) -> +5VD
- U1 pad 2: Net-(C1-Pad1) -> Net-(J6-Pad1)
- U1 pad 3: GND -> Net-(D1-Pad2)
- U1 pad 4: Net-(D1-Pad2) -> GND
- U1 pad 5: Net-(J6-Pad1) -> Net-(C1-Pad1)
- U1 pad 6: +5VD -> Net-(J3-Pad2)
Routing:
- net Net-(J3-Pad2): track 45.4 -> 31.5 mm
- net Net-(J6-Pad1): track 13.8 -> 20.7 mm
- net Net-(J3-Pad1): track 22.8 -> 28.5 mm
- net +5VD: track 18.9 -> 22.7 mm
- net GND: track 14.5 -> 11.4 mm
- net Net-(D1-Pad2): track 9.78 -> 7.55 mm
- net Net-(JP1-Pad2): track 2.09 -> 2.75 mm
- net Net-(JP2-Pad2): track 2.73 -> 2.07 mm
Other:
- board text added: "power heater TPS61165 2/2022"
- board text removed: "power heater TPS61165 10/2021"
