File: TPS61165-heater-v2/TPS61165-heater-v2.sch (KiCad schematic (older format))
At the start: 20 parts, among them J1 USB_C_KoreanHroparts_6P, J2 A2001WV-2P, J3 Conn_01x02_Female, J4 A2001WV-2P, J5 MMCX, J6 Conn_01x02_Female, J7 MMCX, U1 TPS61165

Commit message: Update github
Parts:
- U1: symbol 0JLC:TPS61165 -> 0JLC:TPS61165_SOT
Connections:
- net +5VD: now also U1.1 (VIN); no longer U1.6 (VIN)
- net GND: now also U1.4 (GND); no longer U1.3 (GND)
- net at J3.2 (Pin_2), J4.2 (-), J7.1 (In)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: now also U1.6 (FB); no longer U1.1 (FB)
- net at U1.2 (CTRL): now also J6.1 (Pin_1); no longer C1.1
- net at D1.2 (A), L1.2: now also U1.3 (SW); no longer U1.4 (SW)
- net at U1.5 (COMP): now also C1.1; no longer J6.1 (Pin_1)
Changed lines of the file:
@@
 $EndDescr
 $Comp
-L 0JLC:TPS61165 U1
+L 0JLC:TPS61165_SOT U1
 U 1 1 61311BD9
 P 3650 3500
