File: diode-readouts/ADS112C04-2ch/2ch-ads.kicad_pcb (KiCad board)
At the start: 2 copper layers, 82 x 50 mm, 87 parts, among them IC1 ADS112C04IPWR, IC2 ADS112C04IPWR, J1 DB9_Female_MountingHoles, J10 MMCX, J2 Conn_01x02, J3 Conn_01x02, J4 A1001WV-S-04P, J5 A1001WV-S-04P, J6 MMCX, J7 MMCX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

Commit message: Update github
Parts:
- added JP1: Jumper_3_Open, Jumper:SolderJumper-3_P1.3mm_Open_RoundedPad1.0x1.5mm, B.Cu at (130.2, 112.2)
- added JP9: Jumper_3_Open, Jumper:SolderJumper-3_P1.3mm_Open_RoundedPad1.0x1.5mm, B.Cu at (130.3, 91.2)
Changed lines of the file:
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@@
     (tracks 740)
     (zones 0)
-    (modules 87)
+    (modules 89)
     (nets 55)
   )
@@
     (add_net VD)
   )
+  (module Jumper:SolderJumper-3_P1.3mm_Open_RoundedPad1.0x1.5mm (layer B.Cu)
+    (at 130.35 91.25)
+    (descr "SMD Solder 3-pad Jumper, 1x1.5mm rounded Pads, 0.3mm gap, open")
+    (tags "solder jumper open")
+    (attr virtual)
+    (fp_text reference JP9 (at 0 1.8) (layer B.SilkS)
+      (effects (font (size 1 1) (thickness 0.15)) (justify mirror))
+    )
+    (fp_text value Jumper_3_Open (at 0 -1.9) (layer B.Fab)
+      (effects (font (size 1 1) (thickness 0.15)) (justify mirror))
+    )
+    (fp_arc (start -1.35 0.3) (end -1.35 1) (angle 90) (layer B.SilkS) (width 0.12))
+    (fp_arc (start -1.35 -0.3) (end -2.05 -0.3) (angle 90) (layer B.SilkS) (width 0.12))
+    (fp_arc (start 1.35 -0.3) (end 1.35 -1) (angle 90) (layer B.SilkS) (width 0.12))
+    (fp_arc (start 1.35 0.3) (end 2.05 0.3) (angle 90) (layer B.SilkS) (width 0.12))
+    (fp_line (start 2.3 -1.25) (end -2.3 -1.25) (layer B.CrtYd) (width 0.05))
+    (fp_line (start 2.3 -1.25) (end 2.3 1.25) (layer B.CrtYd) (width 0.05))
+    (fp_line (start -2.3 1.25) (end -2.3 -1.25) (layer B.CrtYd) (width 0.05))
+    (fp_line (start -2.3 1.25) (end 2.3 1.25) (layer B.CrtYd) (width 0.05))
+    (fp_line (start -1.4 1) (end 1.4 1) (layer B.SilkS) (width 0.12))
+    (fp_line (start 2.05 0.3) (end 2.05 -0.3) (layer B.SilkS) (width 0.12))
+    (fp_line (start 1.4 -1) (end -1.4 -1) (layer B.SilkS) (width 0.12))
+    (fp_line (start -2.05 -0.3) (end -2.05 0.3) (layer B.SilkS) (width 0.12))
+    (fp_line (start -1.2 -1.2) (end -1.5 -1.5) (layer B.SilkS) (width 0.12))
+    (fp_line (start -1.5 -1.5) (end -0.9 -1.5) (layer B.SilkS) (width 0.12))
+    (fp_line (start -1.2 -1.2) (end -0.9 -1.5) (layer B.SilkS) (width 0.12))
+    (pad 2 smd rect (at 0 0) (size 1 1.5) (layers B.Cu B.Mask)
+      (net 53 /Channel1/A1))
+    (pad 3 smd custom (at 1.3 0) (size 1 0.5) (layers B.Cu B.Mask)
+      (net 42 /sda) (zone_connect 2)
+      (options (clearance outline) (anchor rect))
+      (primitives
+        (gr_circle (center 0 -0.25) (end 0.5 -0.25) (width 0))
+        (gr_circle (center 0 0.25) (end 0.5 0.25) (width 0))
+        (gr_poly (pts
+           (xy -0.55 0.75) (xy 0 0.75) (xy 0 -0.75) (xy -0.55 -0.75)) (width 0))
+      ))
+    (pad 1 smd custom (at -1.3 0) (size 1 0.5) (layers B.Cu B.Mask)
+      (net 41 /scl) (zone_connect 2)
+      (options (clearance outline) (anchor rect))
+      (primitives
+        (gr_circle (center 0 -0.25) (end 0.5 -0.25) (width 0))
+        (gr_circle (center 0 0.25) (end 0.5 0.25) (width 0))
+        (gr_poly (pts
+           (xy 0.55 0.75) (xy 0 0.75) (xy 0 -0.75) (xy 0.55 -0.75)) (width 0))
+      ))
+  )
+  (module Jumper:SolderJumper-3_P1.3mm_Open_RoundedPad1.0x1.5mm (layer B.Cu)
+    (at 130.25 112.25)
+    (descr "SMD Solder 3-pad Jumper, 1x1.5mm rounded Pads, 0.3mm gap, open")
+    (tags "solder jumper open")
+    (attr virtual)
+    (fp_text reference JP1 (at 0 1.8) (layer B.SilkS)
+      (effects (font (size 1 1) (thickness 0.15)) (justify mirror))
+    )
+    (fp_text value Jumper_3_Open (at 0 -1.9) (layer B.Fab)
+      (effects (font (size 1 1) (thickness 0.15)) (justify mirror))
+    )
+    (fp_arc (start -1.35 0.3) (end -1.35 1) (angle 90) (layer B.SilkS) (width 0.12))
+    (fp_arc (start -1.35 -0.3) (end -2.05 -0.3) (angle 90) (layer B.SilkS) (width 0.12))
+    (fp_arc (start 1.35 -0.3) (end 1.35 -1) (angle 90) (layer B.SilkS) (width 0.12))
+    (fp_arc (start 1.35 0.3) (end 2.05 0.3) (angle 90) (layer B.SilkS) (width 0.12))
+    (fp_line (start 2.3 -1.25) (end -2.3 -1.25) (layer B.CrtYd) (width 0.05))
+    (fp_line (start 2.3 -1.25) (end 2.3 1.25) (layer B.CrtYd) (width 0.05))
+    (fp_line (start -2.3 1.25) (end -2.3 -1.25) (layer B.CrtYd) (width 0.05))
+    (fp_line (start -2.3 1.25) (end 2.3 1.25) (layer B.CrtYd) (width 0.05))
+    (fp_line (start -1.4 1) (end 1.4 1) (layer B.SilkS) (width 0.12))
+    (fp_line (start 2.05 0.3) (end 2.05 -0.3) (layer B.SilkS) (width 0.12))
+    (fp_line (start 1.4 -1) (end -1.4 -1) (layer B.SilkS) (width 0.12))
+    (fp_line (start -2.05 -0.3) (end -2.05 0.3) (layer B.SilkS) (width 0.12))
+    (fp_line (start -1.2 -1.2) (end -1.5 -1.5) (layer B.SilkS) (width 0.12))
+    (fp_line (start -1.5 -1.5) (end -0.9 -1.5) (layer B.SilkS) (width 0.12))
+    (fp_line (start -1.2 -1.2) (end -0.9 -1.5) (layer B.SilkS) (width 0.12))
+    (pad 2 smd rect (at 0 0) (size 1 1.5) (layers B.Cu B.Mask)
+      (net 50 /Channel0/A1))
+    (pad 3 smd custom (at 1.3 0) (size 1 0.5) (layers B.Cu B.Mask)
+      (net 42 /sda) (zone_connect 2)
+      (options (clearance outline) (anchor rect))
+      (primitives
+        (gr_circle (center 0 -0.25) (end 0.5 -0.25) (width 0))
+        (gr_circle (center 0 0.25) (end 0.5 0.25) (width 0))
+        (gr_poly (pts
+           (xy -0.55 0.75) (xy 0 0.75) (xy 0 -0.75) (xy -0.55 -0.75)) (width 0))
+      ))
+    (pad 1 smd custom (at -1.3 0) (size 1 0.5) (layers B.Cu B.Mask)
+      (net 41 /scl) (zone_connect 2)
+      (options (clearance outline) (anchor rect))
+      (primitives
+        (gr_circle (center 0 -0.25) (end 0.5 -0.25) (width 0))
+        (gr_circle (center 0 0.25) (end 0.5 0.25) (width 0))
+        (gr_poly (pts
+           (xy 0.55 0.75) (xy 0 0.75) (xy 0 -0.75) (xy 0.55 -0.75)) (width 0))
+      ))
+  )
   (module Resistor_SMD:R_0603_1608Metric_Pad1.05x0.95mm_HandSolder (layer F.Cu)
