File: diode-readouts/two-wire-single/two-wire-single.kicad_pcb (KiCad board)
At the start: 4 copper layers, 39 x 19 mm, 28 parts, among them IC2 ADS112C04IPWR, J1 Conn_01x04, J2 JST_SH_Conn_01x04_i2c_horizon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, J3 Conn_01x01_Female

Commit message: Add 47ohms for compatibility with ADS122U04.
Parts:
- added R3: 47, Resistor_SMD:R_0402_1005Metric, F.Cu at (127.7, 94.8)
- added R4: 47, Resistor_SMD:R_0402_1005Metric, F.Cu at (128.4, 93.0)
Connections:
- IC2 pad 15: /sda-tx -> /Channel1/SDA
- IC2 pad 16: /scl-rx -> /Channel1/SCL
- JP14 pad 2: /sda-tx -> /Channel1/SDA
- JP9 pad 2: /scl-rx -> /Channel1/SCL
Routing:
- net /sda-tx: track 21.2 -> 11.3 mm, vias 3 -> 2
- net /Channel1/SDA: track 0.00 -> 8.70 mm, vias 0 -> 1
- net /Channel1/SCL: track 0.00 -> 8.16 mm, vias 0 -> 1
- net /scl-rx: track 19.9 -> 13.2 mm, vias 1 -> 0
Changed lines of the file:
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@@
     (thickness 1.6)
     (drawings 15)
-    (tracks 185)
+    (tracks 189)
     (zones 0)
-    (modules 28)
-    (nets 19)
+    (modules 30)
+    (nets 21)
   )
   (page A4)
@@
   (net 17 /scl-rx)
   (net 18 /sda-tx)
+  (net 19 /Channel1/SCL)
+  (net 20 /Channel1/SDA)
   (net_class Default "This is the default net class."
     (clearance 0.2)
@@
     (add_net /Channel1/I+)
     (add_net /Channel1/I-)
+    (add_net /Channel1/SCL)
+    (add_net /Channel1/SDA)
     (add_net /Channel1/V+)
     (add_net /Channel1/V-)
@@
     (add_net "Net-(C27-Pad2)")
     (add_net VD)
+  )
+  (module Resistor_SMD:R_0402_1005Metric (layer F.Cu)
+    (at 128.415 93.05)
+    (descr "Resistor SMD 0402 (1005 Metric), square (rectangular) end terminal, IPC_7351 nominal, (Body size source: http://www.tortai-tech.com/upload/download/2011102023233369053.pdf), generated with kicad-footprint-generator")
+    (tags resistor)
+    (attr smd)
+    (fp_text reference R4 (at 0 -1.17) (layer F.SilkS)
+      (effects (font (size 1 1) (thickness 0.15)))
+    )
+    (fp_text value 47 (at 0 1.17) (layer F.Fab)
+      (effects (font (size 1 1) (thickness 0.15)))
+    )
+    (fp_text user %R (at 0 0) (layer F.Fab)
+      (effects (font (size 0.25 0.25) (thickness 0.04)))
+    )
+    (fp_line (start 0.93 0.47) (end -0.93 0.47) (layer F.CrtYd) (width 0.05))
+    (fp_line (start 0.93 -0.47) (end 0.93 0.47) (layer F.CrtYd) (width 0.05))
+    (fp_line (start -0.93 -0.47) (end 0.93 -0.47) (layer F.CrtYd) (width 0.05))
+    (fp_line (start -0.93 0.47) (end -0.93 -0.47) (layer F.CrtYd) (width 0.05))
+    (fp_line (start 0.5 0.25) (end -0.5 0.25) (layer F.Fab) (width 0.1))
+    (fp_line (start 0.5 -0.25) (end 0.5 0.25) (layer F.Fab) (width 0.1))
+    (fp_line (start -0.5 -0.25) (end 0.5 -0.25) (layer F.Fab) (width 0.1))
+    (fp_line (start -0.5 0.25) (end -0.5 -0.25) (layer F.Fab) (width 0.1))
+    (pad 2 smd roundrect (at 0.485 0) (size 0.59 0.64) (layers F.Cu F.Paste F.Mask) (roundrect_rratio 0.25)
+      (net 18 /sda-tx))
+    (pad 1 smd roundrect (at -0.485 0) (size 0.59 0.64) (layers F.Cu F.Paste F.Mask) (roundrect_rratio 0.25)
+      (net 20 /Channel1/SDA))
+    (model ${KISYS3DMOD}/Resistor_SMD.3dshapes/R_0402_1005Metric.wrl
+      (at (xyz 0 0 0))
+      (scale (xyz 1 1 1))
+      (rotate (xyz 0 0 0))
+    )
+  )
+  (module Resistor_SMD:R_0402_1005Metric (layer F.Cu)
+    (at 127.665 94.85 180)
+    (descr "Resistor SMD 0402 (1005 Metric), square (rectangular) end terminal, IPC_7351 nominal, (Body size source: http://www.tortai-tech.com/upload/download/2011102023233369053.pdf), generated with kicad-footprint-generator")
+    (tags resistor)
+    (attr smd)
+    (fp_text reference R3 (at 0 -1.17) (layer F.SilkS)
+      (effects (font (size 1 1) (thickness 0.15)))
+    )
+    (fp_text value 47 (at 0 1.17) (layer F.Fab)
+      (effects (font (size 1 1) (thickness 0.15)))
+    )
+    (fp_text user %R (at 0 0) (layer F.Fab)
+      (effects (font (size 0.25 0.25) (thickness 0.04)))
+    )
+    (fp_line (start 0.93 0.47) (end -0.93 0.47) (layer F.CrtYd) (width 0.05))
+    (fp_line (start 0.93 -0.47) (end 0.93 0.47) (layer F.CrtYd) (width 0.05))
+    (fp_line (start -0.93 -0.47) (end 0.93 -0.47) (layer F.CrtYd) (width 0.05))
+    (fp_line (start -0.93 0.47) (end -0.93 -0.47) (layer F.CrtYd) (width 0.05))
+    (fp_line (start 0.5 0.25) (end -0.5 0.25) (layer F.Fab) (width 0.1))
+    (fp_line (start 0.5 -0.25) (end 0.5 0.25) (layer F.Fab) (width 0.1))
+    (fp_line (start -0.5 -0.25) (end 0.5 -0.25) (layer F.Fab) (width 0.1))
+    (fp_line (start -0.5 0.25) (end -0.5 -0.25) (layer F.Fab) (width 0.1))
+    (pad 2 smd roundrect (at 0.485 0 180) (size 0.59 0.64) (layers F.Cu F.Paste F.Mask) (roundrect_rratio 0.25)
+      (net 19 /Channel1/SCL))
+    (pad 1 smd roundrect (at -0.485 0 180) (size 0.59 0.64) (layers F.Cu F.Paste F.Mask) (roundrect_rratio 0.25)
+      (net 17 /scl-rx))
+    (model ${KISYS3DMOD}/Resistor_SMD.3dshapes/R_0402_1005Metric.wrl
+      (at (xyz 0 0 0))
+      (scale (xyz 1 1 1))
+      (rotate (xyz 0 0 0))
+    )
   )
   (module Connector_PinSocket_2.54mm:PinSocket_1x01_P2.54mm_Vertical (layer F.Cu)
@@
     (fp_line (start -1.2 -1.2) (end -0.9 -1.5) (layer B.SilkS) (width 0.12))
     (pad 2 smd rect (at 0 0) (size 1 1.5) (layers B.Cu B.Mask)
-      (net 17 /scl-rx))
+      (net 19 /Channel1/SCL))
     (pad 3 smd custom (at 1.3 0) (size 1 0.5) (layers B.Cu B.Mask)
       (net 13 /Channel1/A1) (zone_connect 2)
@@
     (fp_line (start -1.2 -1.2) (end -0.9 -1.5) (layer B.SilkS) (width 0.12))
     (pad 2 smd rect (at 0 0) (size 1 1.5) (layers B.Cu B.Mask)
-      (net 18 /sda-tx))
+      (net 20 /Channel1/SDA))
     (pad 3 smd custom (at 1.3 0) (size 1 0.5) (layers B.Cu B.Mask)
       (net 13 /Channel1/A1) (zone_connect 2)
@@
     (fp_line (start -1.2 -2.5) (end 2.2 -2.5) (layer F.Fab) (width 0.15))
     (pad 16 smd rect (at 2.95 -2.275 270) (size 1.5 0.45) (layers F.Cu F.Paste F.Mask)
-      (net 17 /scl-rx))
+      (net 19 /Channel1/SCL))
     (pad 15 smd rect (at 2.95 -1.625 270) (size 1.5 0.45) (layers F.Cu F.Paste F.Mask)
-      (net 18 /sda-tx))
+      (net 20 /Channel1/SDA))
     (pad 14 smd rect (at 2.95 -0.975 270) (size 1.5 0.45) (layers F.Cu F.Paste F.Mask)
       (net 15 /Channel1/~DRDY))
@@
   (segment (start 120.1 91.75) (end 120.1 86.9) (width 0.25) (layer In1.Cu) (net 15))
   (segment (start 135.650001 96.563189) (end 134.56319 97.65) (width 0.25) (layer F.Cu) (net 16))
-  (via (at 127.15 96.05) (size 0.6) (drill 0.4) (layers F.Cu B.Cu) (net 17))
-  (segment (start 121.9 93.1) (end 124.85 96.05) (width 0.25) (layer F.Cu) (net 17))
-  (segment (start 124.85 96.05) (end 127.15 96.05) (width 0.25) (layer F.Cu) (net 17))
-  (segment (start 121.425 93.1) (end 121.9 93.1) (width 0.25) (layer F.Cu) (net 17))
-  (segment (start 127.15 96.05) (end 128.4 96.05) (width 0.25) (layer F.Cu) (net 17))
-  (segment (start 130.4 94.5) (end 130.175 94.275) (width 0.25) (layer F.Cu) (net 17))
+  (via (at 127.15 96.05) (size 0.6) (drill 0.4) (layers F.Cu B.Cu) (net 19))
+  (segment (start 121.9 93.1) (end 124.85 96.05) (width 0.25) (layer F.Cu) (net 19))
+  (segment (start 124.85 96.05) (end 127.15 96.05) (width 0.25) (layer F.Cu) (net 19))
+  (segment (start 121.425 93.1) (end 121.9 93.1) (width 0.25) (layer F.Cu) (net 19))
   (segment (start 130.4 95.625) (end 130.4 94.5) (width 0.25) (layer F.Cu) (net 17))
-  (segment (start 128.4 96.05) (end 130.175 94.275) (width 0.25) (layer F.Cu) (net 17))
   (segment (start 130.22501 90.77499) (end 130.22501 94.22499) (width 0.25) (layer F.Cu) (net 17))
-  (segment (start 130.22501 94.22499) (end 130.175 94.275) (width 0.25) (layer F.Cu) (net 17))
   (segment (start 132 89) (end 130.22501 90.77499) (width 0.25) (layer F.Cu) (net 17))
   (segment (start 133.75 89) (end 132 89) (width 0.25) (layer F.Cu) (net 17))
-  (segment (start 120.775 92.189998) (end 121.114998 91.85) (width 0.25) (layer F.Cu) (net 18))
-  (segment (start 120.775 93.1) (end 120.775 92.189998) (width 0.25) (layer F.Cu) (net 18))
-  (segment (start 121.114998 91.85) (end 122.05 91.85) (width 0.25) (layer F.Cu) (net 18))
-  (segment (start 123.25 93.05) (end 127.15 93.05) (width 0.25) (layer F.Cu) (net 18))
-  (via (at 127.15 93.05) (size 0.6) (drill 0.4) (layers F.Cu B.Cu) (net 18))
-  (segment (start 122.05 91.85) (end 123.25 93.05) (width 0.25) (layer F.Cu) (net 18))
-  (segment (start 127.15 93.05) (end 129.775 93.05) (width 0.25) (layer F.Cu) (net 18))
+  (segment (start 130.4 95.1) (end 130.4 95.625) (width 0.25) (layer F.Cu) (net 17))
+  (segment (start 130.15 94.85) (end 130.4 95.1) (width 0.25) (layer F.Cu) (net 17))
+  (segment (start 128.15 94.85) (end 130.15 94.85) (width 0.25) (layer F.Cu) (net 17))
+  (segment (start 130.4 94.39998) (end 130.4 95.625) (width 0.25) (layer F.Cu) (net 17))
+  (segment (start 130.22501 94.22499) (end 130.4 94.39998) (width 0.25) (layer F.Cu) (net 17))
+  (segment (start 120.775 92.189998) (end 121.114998 91.85) (width 0.25) (layer F.Cu) (net 20))
+  (segment (start 120.775 93.1) (end 120.775 92.189998) (width 0.25) (layer F.Cu) (net 20))
+  (segment (start 121.114998 91.85) (end 122.05 91.85) (width 0.25) (layer F.Cu) (net 20))
+  (segment (start 123.25 93.05) (end 127.15 93.05) (width 0.25) (layer F.Cu) (net 20))
+  (via (at 127.15 93.05) (size 0.6) (drill 0.4) (layers F.Cu B.Cu) (net 20))
+  (segment (start 122.05 91.85) (end 123.25 93.05) (width 0.25) (layer F.Cu) (net 20))
   (via (at 130.85001 93.05) (size 0.6) (drill 0.4) (layers F.Cu B.Cu) (net 18))
   (segment (start 130.85001 90.87501) (end 130.85001 93.05) (width 0.25) (layer F.Cu) (net 18))
@@
   (segment (start 131.72502 90) (end 130.85001 90.87501) (width 0.25) (layer F.Cu) (net 18))
   (segment (start 133.75 90) (end 131.72502 90) (width 0.25) (layer F.Cu) (net 18))
+  (segment (start 128.9 93.05) (end 129.60001 93.05) (width 0.25) (layer F.Cu) (net 18))
+  (segment (start 127.15 94.88) (end 127.18 94.85) (width 0.25) (layer F.Cu) (net 19))
+  (segment (start 127.15 96.05) (end 127.15 94.88) (width 0.25) (layer F.Cu) (net 19))
+  (segment (start 127.93 93.05) (end 127.15 93.05) (width 0.25) (layer F.Cu) (net 20))
   (zone (net 1) (net_name GND) (layer F.Cu) (hatch edge 0.508)
     (connect_pads (clearance 0.508))
