File: ADC circuits/sq_lockin_v3/2opamp.sch (KiCad schematic (older format))
At the start: 4 parts, among them U5 LMP7715, U6 LMP7715

Commit message: Add power-two-wre and tweaks to sq_lockin_v3
Changed lines of the file:
@@
 AR Path="/621A3D17/621A90E2" Ref="U5"  Part="1"
 AR Path="/624D2E5E/621A90E2" Ref="U9"  Part="1"
-F 0 "U9" H 4750 4000 50  0000 C CNN
+F 0 "U5" H 4750 4000 50  0000 C CNN
 F 1 "LMP7715" H 4900 3850 50  0000 C CNN
 F 2 "Package_TO_SOT_SMD:TSOT-23-5" H 4750 4000 50  0001 C CNN
@@
 AR Path="/621A3D17/621A90F6" Ref="#PWR0112"  Part="1"
 AR Path="/624D2E5E/621A90F6" Ref="#PWR0102"  Part="1"
-F 0 "#PWR0102" H 4650 4050 50  0001 C CNN
+F 0 "#PWR0112" H 4650 4050 50  0001 C CNN
 F 1 "GND" V 4655 4172 50  0000 R CNN
 F 2 "" H 4650 4300 50  0001 C CNN
@@
 AR Path="/621A3D17/621A9105" Ref="C8"  Part="1"
 AR Path="/624D2E5E/621A9105" Ref="C10"  Part="1"
-F 0 "C10" V 4548 3700 50  0000 C CNN
+F 0 "C8" V 4548 3700 50  0000 C CNN
 F 1 "100nF" V 4639 3700 50  0000 C CNN
 F 2 "Capacitor_SMD:C_0603_1608Metric_Pad1.05x0.95mm_HandSolder" H 4838 3550 50  0001 C CNN
@@
 AR Path="/621A3D17/621A910B" Ref="#PWR0114"  Part="1"
 AR Path="/624D2E5E/621A910B" Ref="#PWR0103"  Part="1"
-F 0 "#PWR0103" H 4950 3450 50  0001 C CNN
+F 0 "#PWR0114" H 4950 3450 50  0001 C CNN
 F 1 "GND" V 4955 3572 50  0000 R CNN
 F 2 "" H 4950 3700 50  0001 C CNN
@@
 AR Path="/621A3D17/621A9117" Ref="#PWR0115"  Part="1"
 AR Path="/624D2E5E/621A9117" Ref="#PWR0104"  Part="1"
-F 0 "#PWR0104" H 4350 3450 50  0001 C CNN
+F 0 "#PWR0115" H 4350 3450 50  0001 C CNN
 F 1 "VCC" H 4367 3773 50  0000 C CNN
 F 2 "" H 4350 3600 50  0001 C CNN
@@
 AR Path="/621A3D17/621B016B" Ref="U6"  Part="1"
 AR Path="/624D2E5E/621B016B" Ref="U10"  Part="1"
-F 0 "U10" H 4750 5250 50  0000 C CNN
+F 0 "U6" H 4750 5250 50  0000 C CNN
 F 1 "LMP7715" H 4900 5100 50  0000 C CNN
 F 2 "Package_TO_SOT_SMD:TSOT-23-5" H 4750 5250 50  0001 C CNN
@@
 AR Path="/621A3D17/621B0176" Ref="#PWR0116"  Part="1"
 AR Path="/624D2E5E/621B0176" Ref="#PWR0107"  Part="1"
-F 0 "#PWR0107" H 4650 5300 50  0001 C CNN
+F 0 "#PWR0116" H 4650 5300 50  0001 C CNN
 F 1 "GND" V 4655 5422 50  0000 R CNN
 F 2 "" H 4650 5550 50  0001 C CNN
@@
 AR Path="/621A3D17/621B017E" Ref="C9"  Part="1"
 AR Path="/624D2E5E/621B017E" Ref="C11"  Part="1"
-F 0 "C11" V 4548 4950 50  0000 C CNN
+F 0 "C9" V 4548 4950 50  0000 C CNN
 F 1 "100nF" V 4639 4950 50  0000 C CNN
 F 2 "Capacitor_SMD:C_0603_1608Metric_Pad1.05x0.95mm_HandSolder" H 4838 4800 50  0001 C CNN
@@
 AR Path="/621A3D17/621B0184" Ref="#PWR0121"  Part="1"
 AR Path="/624D2E5E/621B0184" Ref="#PWR0109"  Part="1"
-F 0 "#PWR0109" H 4950 4700 50  0001 C CNN
+F 0 "#PWR0121" H 4950 4700 50  0001 C CNN
 F 1 "GND" V 4955 4822 50  0000 R CNN
 F 2 "" H 4950 4950 50  0001 C CNN
@@
 AR Path="/621A3D17/621B018C" Ref="#PWR0122"  Part="1"
 AR Path="/624D2E5E/621B018C" Ref="#PWR0111"  Part="1"
-F 0 "#PWR0111" H 4350 4700 50  0001 C CNN
+F 0 "#PWR0122" H 4350 4700 50  0001 C CNN
 F 1 "VCC" H 4367 5023 50  0000 C CNN
 F 2 "" H 4350 4850 50  0001 C CNN
