File: ADC circuits/sq_lockin_v3/IA.sch (KiCad schematic (older format))
At the start: 14 parts, among them J17 Conn_01x02_Male_2.54mm, J18 Conn_01x02_Male_2.54mm, U10 AD623, U11 LMP7715, U8 LMP7715, U9 LMP7715

Commit message: Add power-two-wre and tweaks to sq_lockin_v3
Parts:
- removed J17, J18: Conn_01x02_Male_2.54mm, Connector_PinHeader_2.54mm:PinHeader_1x02_P2.54mm_Vertical, symbol 0JLC:Conn_01x02_Male_2.54mm
- removed R3: DNF, Resistor_SMD:R_0603_1608Metric_Pad1.05x0.95mm_HandSolder, symbol 0JLC:R
- added J13: Conn_01x02_Male_2.54mm, Connector_PinHeader_2.54mm:PinHeader_1x02_P2.54mm_Vertical, symbol 0JLC:Conn_01x02_Male_2.54mm
- added R25: 100, Resistor_SMD:R_0603_1608Metric_Pad1.05x0.95mm_HandSolder, symbol 0JLC:100
Connections:
- net labels added: in+, in-, out+, out-
- wire segments 60 -> 58
