File: ADC circuits/sq_lockin_v3/polarity_inverter.sch (KiCad schematic (older format))
At the start: 9 parts, among them J12 Conn_01x02_Male_2.54mm, Q1 BSS84, Q2 2N7002, U7 AQW212EHAX, U8 AQW212EHAX

Commit message: Add power-two-wre and tweaks to sq_lockin_v3
Parts:
- removed J12: Conn_01x02_Male_2.54mm, Connector_PinHeader_2.54mm:PinHeader_1x02_P2.54mm_Vertical, symbol 0JLC:Conn_01x02_Male_2.54mm
Connections:
- net ctrl-: now also Q1.3 (D), Q2.3 (D)
Changed lines of the file:
@@
 $Descr A4 11693 8268
 encoding utf-8
-Sheet 4 8
+Sheet 7 8
 Title ""
 Date ""
@@
 AR Path="/624D2E6E/624B66C6" Ref="U13"  Part="1"
 AR Path="/6256EE34/624B66C6" Ref="U16"  Part="1"
-F 0 "U7" H 5400 3575 50  0000 C CNN
+F 0 "U16" H 5400 3575 50  0000 C CNN
 F 1 "AQW212EHAX" H 5400 3484 50  0000 C CNN
 F 2 "0my_footprints:SMD-8_L9.8-W6.4-P2.54-LS10.0-BL" H 5200 3050 50  0001 L CIN
@@
 AR Path="/624D2E6E/624B66CC" Ref="U13"  Part="2"
 AR Path="/6256EE34/624B66CC" Ref="U16"  Part="2"
-F 0 "U7" H 5400 4125 50  0000 C CNN
+F 0 "U16" H 5400 4125 50  0000 C CNN
 F 1 "AQW212EHAX" H 5400 4034 50  0000 C CNN
 F 2 "0my_footprints:SMD-8_L9.8-W6.4-P2.54-LS10.0-BL" H 5200 3600 50  0001 L CIN
@@
 AR Path="/624D2E6E/624B66D2" Ref="U14"  Part="1"
 AR Path="/6256EE34/624B66D2" Ref="U17"  Part="1"
-F 0 "U8" H 6550 3575 50  0000 C CNN
+F 0 "U17" H 6550 3575 50  0000 C CNN
 F 1 "AQW212EHAX" H 6550 3484 50  0000 C CNN
 F 2 "0my_footprints:SMD-8_L9.8-W6.4-P2.54-LS10.0-BL" H 6350 3050 50  0001 L CIN
@@
 AR Path="/624D2E6E/624B66D8" Ref="U14"  Part="2"
 AR Path="/6256EE34/624B66D8" Ref="U17"  Part="2"
-F 0 "U8" H 6550 4125 50  0000 C CNN
+F 0 "U17" H 6550 4125 50  0000 C CNN
 F 1 "AQW212EHAX" H 6550 4034 50  0000 C CNN
 F 2 "0my_footprints:SMD-8_L9.8-W6.4-P2.54-LS10.0-BL" H 6350 3600 50  0001 L CIN
@@
 AR Path="/624D2E6E/624B66EA" Ref="R15"  Part="1"
 AR Path="/6256EE34/624B66EA" Ref="R21"  Part="1"
-F 0 "R3" V 4743 3150 50  0000 C CNN
+F 0 "R21" V 4743 3150 50  0000 C CNN
 F 1 "200" V 4834 3150 50  0000 C CNN
 F 2 "Resistor_SMD:R_0603_1608Metric_Pad1.05x0.95mm_HandSolder" V 4880 3150 50  0001 C CNN
@@
 AR Path="/624D2E6E/624B66F7" Ref="R16"  Part="1"
 AR Path="/6256EE34/624B66F7" Ref="R22"  Part="1"
-F 0 "R4" V 4743 3700 50  0000 C CNN
+F 0 "R22" V 4743 3700 50  0000 C CNN
 F 1 "200" V 4834 3700 50  0000 C CNN
 F 2 "Resistor_SMD:R_0603_1608Metric_Pad1.05x0.95mm_HandSolder" V 4880 3700 50  0001 C CNN
@@
 AR Path="/624D2E6E/624B6703" Ref="R19"  Part="1"
 AR Path="/6256EE34/624B6703" Ref="R23"  Part="1"
-F 0 "R6" V 6793 3150 50  0000 C CNN
+F 0 "R23" V 6793 3150 50  0000 C CNN
 F 1 "200" V 6884 3150 50  0000 C CNN
 F 2 "Resistor_SMD:R_0603_1608Metric_Pad1.05x0.95mm_HandSolder" V 6930 3150 50  0001 C CNN
@@
 AR Path="/624D2E6E/624B6711" Ref="R20"  Part="1"
 AR Path="/6256EE34/624B6711" Ref="R24"  Part="1"
-F 0 "R7" V 6793 3700 50  0000 C CNN
+F 0 "R24" V 6793 3700 50  0000 C CNN
 F 1 "200" V 6884 3700 50  0000 C CNN
 F 2 "Resistor_SMD:R_0603_1608Metric_Pad1.05x0.95mm_HandSolder" V 6930 3700 50  0001 C CNN
@@
 AR Path="/624D2E6E/62443B5E" Ref="Q4"  Part="1"
 AR Path="/6256EE34/62443B5E" Ref="Q6"  Part="1"
-F 0 "Q2" H 3854 4746 50  0000 L CNN
+F 0 "Q6" H 3854 4746 50  0000 L CNN
 F 1 "2N7002" H 3854 4655 50  0000 L CNN
 F 2 "Package_TO_SOT_SMD:SOT-23" H 3850 4625 50  0001 L CIN
@@
 AR Path="/624D2E6E/62447052" Ref="Q3"  Part="1"
 AR Path="/6256EE34/62447052" Ref="Q5"  Part="1"
-F 0 "Q1" H 3854 4104 50  0000 L CNN
+F 0 "Q5" H 3854 4104 50  0000 L CNN
 F 1 "BSS84" H 3854 4195 50  0000 L CNN
 F 2 "Package_TO_SOT_SMD:SOT-23" H 3850 4075 50  0001 L CIN
@@
 AR Path="/624D2E6E/6244B7D9" Ref="#PWR0126"  Part="1"
 AR Path="/6256EE34/6244B7D9" Ref="#PWR0131"  Part="1"
-F 0 "#PWR0105" H 3750 4700 50  0001 C CNN
+F 0 "#PWR0131" H 3750 4700 50  0001 C CNN
 F 1 "GND" H 3755 4777 50  0000 C CNN
 F 2 "" H 3750 4950 50  0001 C CNN
@@
 AR Path="/624D2E6E/6244D68A" Ref="#PWR0130"  Part="1"
 AR Path="/6256EE34/6244D68A" Ref="#PWR0132"  Part="1"
-F 0 "#PWR0106" H 3750 3750 50  0001 C CNN
+F 0 "#PWR0132" H 3750 3750 50  0001 C CNN
 F 1 "VCC" H 3767 4073 50  0000 C CNN
 F 2 "" H 3750 3900 50  0001 C CNN
@@
 	1    0    0    -1
 $EndComp
-$Comp
-L 0JLC:Conn_01x02_Male_2.54mm J12
-U 1 1 6246BB5F
-P 4300 4400
-AR Path="/624B5D4F/6246BB5F" Ref="J12"  Part="1"
-AR Path="/624D2E6E/6246BB5F" Ref="J13"  Part="1"
-AR Path="/6256EE34/6246BB5F" Ref="J14"  Part="1"
-F 0 "J12" H 4272 4282 50  0000 R CNN
-F 1 "Conn_01x02_Male_2.54mm" H 4272 4373 50  0000 R CNN
-F 2 "Connector_PinHeader_2.54mm:PinHeader_1x02_P2.54mm_Vertical" H 4300 4400 50  0001 C CNN
-F 3 "~" H 4300 4400 50  0001 C CNN
-F 4 "C492401" H 4300 4400 50  0001 C CNN "LCSC"
-F 5 "PZ254V-11-02P" H 4300 4400 50  0001 C CNN "MPN"
-	1    4300 4400
-	-1   0    0    1
-$EndComp
 Wire Wire Line
 	3750 4450 4100 4450
-Wire Wire Line
-	4100 4450 4100 4400
 Connection ~ 3750 4450
 Wire Wire Line
 	3750 4450 3750 4500
-Wire Wire Line
-	4100 4300 4100 3700
 Connection ~ 4100 3700
 Wire Wire Line
@@
 Wire Wire Line
 	3450 4450 3450 4700
+Wire Wire Line
+	4100 3700 4100 4450
 $EndSCHEMATC
