File: TPS61165-heater/TPS61165-heater.sch (KiCad schematic (older format))
At the start: 24 parts, among them J1 USB_C_KoreanHroparts_6P, J2 A2001WV-2P, J3 Conn_01x02_Female, J4 A2001WV-2P, J5 MMCX, J6 Conn_01x03_Female, J7 A1001WV-S-04P, U1 TPS61165, U2 KAQY212A, U3 INA226

Commit message: Add power-two-wre and tweaks to sq_lockin_v3
Parts:
- U1: symbol 0JLC:TPS61165 -> TPS61165-heater-rescue:TPS61165-0JLC
Changed lines of the file:
@@
 $EndDescr
 $Comp
-L 0JLC:TPS61165 U1
+L TPS61165-heater-rescue:TPS61165-0JLC U1
 U 1 1 61311BD9
 P 3650 3500
