File: diode-readouts/power-two-wire/power-two-wire.kicad_pcb (KiCad board)
At the start: 2 copper layers, 45 x 50 mm, 38 parts, among them J1 JST_SH_Conn_01x04_i2c_horizon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, J2 JST_SH_Conn_01x04_i2c_horizon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, J3 JST_SH_Conn_01x04_i2c_horizon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, J4 A1001WV-S-04P, J5 A1001WV-S-04P, J6 JST_SH_Conn_01x04_i2c_horizon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, J7 Conn_01x06_SPI, J8 Conn_01x06_Female, J9 MMCX, Q1 BC847C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

Commit message: add uart mux versions
Connections:
- C1 pad 1: /Sheet605654E7/i2c_power -> VCC
- L1 pad 2: /Sheet605654E7/i2c_power -> VCC
Routing:
- net VCC: track 23.6 -> 35.5 mm
- net /Sheet605654E7/i2c_power: track 5.53 -> 0.00 mm
