File: uart_mux_v1/power.sch (KiCad schematic (older format))
At the start: 19 parts, among them J9 MMCX, Q1 BC847C, U1 LP5907MFX-3.3, U2 LP5907MFX-3.3

Commit message: add uart mux versions
Parts:
- removed C7, C9: 1uF, Capacitor_SMD:C_0603_1608Metric_Pad1.05x0.95mm_HandSolder, symbol 0JLC:1uF
- removed JP2, JP3: Jumper_NO_Small, Jumper:SolderJumper-2_P1.3mm_Open_Pad1.0x1.5mm, symbol Device:Jumper_NO_Small
- removed U2: LP5907MFX-3.3, Package_TO_SOT_SMD:SOT-23-5, symbol 0JLC:LP5907MFX-3.3
- renumbered C1 to C2, C2 to C3, C3 to C4, C4 to C5, C5 to C6, C6 to C7, C8 to C9, J9 to J7, U1 to U2
Connections:
- net labels added: gnd_in, power_in
- net labels removed: VCC, digital, i2c_power
- wire segments 64 -> 48
Changed lines of the file:
@@
 analog
 $Comp
-L Device:C C3
+L Device:C C4
 U 1 1 605729C4
 P 5100 4150
-F 0 "C3" H 5125 4250 50  0000 L CNN
+F 0 "C4" H 5125 4250 50  0000 L CNN
 F 1 "100nF" H 5250 4200 50  0000 L TNN
 F 2 "Capacitor_SMD:C_0603_1608Metric_Pad1.05x0.95mm_HandSolder" H 5138 4000 50  0001 C CNN
@@
 $EndComp
 $Comp
-L Device:C C4
+L Device:C C5
 U 1 1 605729CF
 P 5700 4150
-F 0 "C4" H 5725 4250 50  0000 L CNN
+F 0 "C5" H 5725 4250 50  0000 L CNN
 F 1 "10nF" H 5850 4200 50  0000 L TNN
 F 2 "Capacitor_SMD:C_0603_1608Metric_Pad1.05x0.95mm_HandSolder" H 5738 4000 50  0001 C CNN
@@
 $EndComp
 $Comp
-L power:GND #PWR0104
+L power:GND #PWR016
 U 1 1 605729DD
 P 5700 4400
-F 0 "#PWR0104" H 5700 4150 50  0001 C CNN
+F 0 "#PWR016" H 5700 4150 50  0001 C CNN
 F 1 "GND" H 5700 4250 50  0000 C CNN
 F 2 "" H 5700 4400 50  0001 C CNN
@@
 	6800 4300 6800 4350
 $Comp
-L power:GND #PWR0106
+L power:GND #PWR017
 U 1 1 60580F4B
 P 6800 4700
-F 0 "#PWR0106" H 6800 4450 50  0001 C CNN
+F 0 "#PWR017" H 6800 4450 50  0001 C CNN
 F 1 "GND" H 6800 4550 50  0000 C CNN
 F 2 "" H 6800 4700 50  0001 C CNN
@@
 Text HLabel 10150 4000 2    50   Output ~ 0
 analog
-Wire Wire Line
-	7700 4000 7750 4000
 $Comp
 L 0my_power:B0305S-1WR2 PS1
@@
 	1    0    0    -1
 $EndComp
-Text Label 2450 4000 2    50   ~ 0
-i2c_power
 $Comp
 L pspice:INDUCTOR L1
@@
 $EndComp
 $Comp
-L power:GNDPWR #PWR0107
+L power:GNDPWR #PWR015
 U 1 1 60EB8126
 P 2550 4400
-F 0 "#PWR0107" H 2550 4200 50  0001 C CNN
+F 0 "#PWR015" H 2550 4200 50  0001 C CNN
 F 1 "GNDPWR" H 2554 4246 50  0000 C CNN
 F 2 "" H 2550 4350 50  0001 C CNN
@@
 $EndComp
 $Comp
-L 0JLC:10uF_1206_50V C2
+L 0JLC:10uF_1206_50V C3
 U 1 1 60EBDADE
 P 4450 4150
-F 0 "C2" H 4550 4100 50  0000 L CNN
+F 0 "C3" H 4550 4100 50  0000 L CNN
 F 1 "10uF_1206_50V" H 4500 4250 50  0000 L CNN
 F 2 "Capacitor_SMD:C_1206_3216Metric_Pad1.42x1.75mm_HandSolder" H 4488 4000 50  0001 C CNN
@@
 $EndComp
 $Comp
-L 0JLC:4.7uF_1206_50V C1
+L 0JLC:4.7uF_1206_50V C2
 U 1 1 60EBE33B
 P 2550 4150
-F 0 "C1" H 2665 4196 50  0000 L CNN
+F 0 "C2" H 2665 4196 50  0000 L CNN
 F 1 "4.7uF_1206_50V" H 2665 4105 50  0000 L CNN
 F 2 "Capacitor_SMD:C_1206_3216Metric_Pad1.42x1.75mm_HandSolder" H 2588 4000 50  0001 C CNN
@@
 $EndComp
 $Comp
-L Device:CP C5
+L Device:CP C6
 U 1 1 60EC45A8
 P 6800 4550
-F 0 "C5" H 6915 4596 50  0000 L CNN
+F 0 "C6" H 6915 4596 50  0000 L CNN
 F 1 "100uF" H 6915 4505 50  0000 L CNN
 F 2 "Capacitor_Tantalum_SMD:CP_EIA-3528-12_Kemet-T" H 6838 4400 50  0001 C CNN
@@
 Connection ~ 4450 4300
 $Comp
-L 0JLC:LP5907MFX-3.3 U1
+L 0JLC:LP5907MFX-3.3 U2
 U 1 1 60EC7284
 P 8750 4100
-F 0 "U1" H 8750 4467 50  0000 C CNN
+F 0 "U2" H 8750 4467 50  0000 C CNN
 F 1 "LP5907MFX-3.3" H 8750 4376 50  0000 C CNN
 F 2 "Package_TO_SOT_SMD:SOT-23-5" H 8750 4450 50  0001 C CNN
@@
 Wire Wire Line
 	8350 4000 8450 4000
-Wire Wire Line
-	7750 4950 8200 4950
-$Comp
-L 0JLC:LP5907MFX-3.3 U2
-U 1 1 60ECAF07
-P 8800 5050
-F 0 "U2" H 8800 5417 50  0000 C CNN
-F 1 "LP5907MFX-3.3" H 8800 5326 50  0000 C CNN
-F 2 "Package_TO_SOT_SMD:SOT-23-5" H 8800 5400 50  0001 C CNN
-F 3 "http://www.ti.com/lit/ds/symlink/lp5907.pdf" H 8800 5550 50  0001 C CNN
-F 4 "C80670" H 8800 5050 50  0001 C CNN "LCSC"
-F 5 "LP5907MFX-3.3/NOPB" H 8800 5050 50  0001 C CNN "MPN"
-	1    8800 5050
-	1    0    0    -1
-$EndComp
-Wire Wire Line
-	8800 5350 8800 5500
-Wire Wire Line
-	8800 5500 9250 5500
-Wire Wire Line
-	8400 4950 8400 5050
-Wire Wire Line
-	8400 5050 8500 5050
-Connection ~ 8400 4950
-Wire Wire Line
-	8400 4950 8500 4950
-Wire Wire Line
-	7750 4000 7750 4950
-Connection ~ 7750 4000
-Wire Wire Line
-	7750 4000 7950 4000
 $Comp
 L 0JLC:1uF C7
-U 1 1 60ECCAB0
-P 8200 5100
-F 0 "C7" H 8315 5146 50  0000 L CNN
-F 1 "1uF" H 8315 5055 50  0000 L CNN
-F 2 "Capacitor_SMD:C_0603_1608Metric_Pad1.05x0.95mm_HandSolder" H 8238 4950 50  0001 C CNN
-F 3 "~" H 8200 5100 50  0001 C CNN
-F 4 "C15849" H 8200 5100 50  0001 C CNN "LCSC"
-F 5 "CL10A105KB8NNNC" H 8200 5100 50  0001 C CNN "MPN"
-	1    8200 5100
-	1    0    0    -1
-$EndComp
-Connection ~ 8200 4950
-Wire Wire Line
-	8200 4950 8400 4950
-$Comp
-L 0JLC:1uF C6
 U 1 1 60ECD8E2
 P 8150 4150
-F 0 "C6" H 8265 4196 50  0000 L CNN
+F 0 "C7" H 8265 4196 50  0000 L CNN
 F 1 "1uF" H 8265 4105 50  0000 L CNN
 F 2 "Capacitor_SMD:C_0603_1608Metric_Pad1.05x0.95mm_HandSolder" H 8188 4000 50  0001 C CNN
@@
 	8150 4000 8350 4000
 $Comp
-L 0JLC:1uF C8
+L 0JLC:1uF C9
 U 1 1 60ECDE32
 P 9250 4150
-F 0 "C8" H 9365 4196 50  0000 L CNN
+F 0 "C9" H 9365 4196 50  0000 L CNN
 F 1 "1uF" H 9365 4105 50  0000 L CNN
 F 2 "Capacitor_SMD:C_0603_1608Metric_Pad1.05x0.95mm_HandSolder" H 9288 4000 50  0001 C CNN
@@
 	1    0    0    -1
 $EndComp
-$Comp
-L 0JLC:1uF C9
-U 1 1 60ECE60A
-P 9250 5100
-F 0 "C9" H 9365 5146 50  0000 L CNN
-F 1 "1uF" H 9365 5055 50  0000 L CNN
-F 2 "Capacitor_SMD:C_0603_1608Metric_Pad1.05x0.95mm_HandSolder" H 9288 4950 50  0001 C CNN
-F 3 "~" H 9250 5100 50  0001 C CNN
-F 4 "C15849" H 9250 5100 50  0001 C CNN "LCSC"
-F 5 "CL10A105KB8NNNC" H 9250 5100 50  0001 C CNN "MPN"
-	1    9250 5100
-	1    0    0    -1
-$EndComp
-Wire Wire Line
-	9250 5250 9250 5500
-Connection ~ 9250 5500
-Wire Wire Line
-	9250 5500 9350 5500
 Wire Wire Line
 	9250 4300 9250 4550
@@
 Wire Wire Line
 	9250 4000 9050 4000
-Wire Wire Line
-	9100 4950 9250 4950
-Wire Wire Line
-	8800 5500 8200 5500
-Wire Wire Line
-	8200 5500 8200 5250
-Connection ~ 8800 5500
 Wire Wire Line
 	8750 4550 8150 4550
@@
 	9250 4000 9250 3800
 $Comp
-L power:GND #PWR0108
+L power:GND #PWR018
 U 1 1 60ED5D4E
 P 9300 4550
-F 0 "#PWR0108" H 9300 4300 50  0001 C CNN
+F 0 "#PWR018" H 9300 4300 50  0001 C CNN
 F 1 "GND" H 9300 4400 50  0000 C CNN
 F 2 "" H 9300 4550 50  0001 C CNN
@@
 	1    0    0    -1
 $EndComp
-$Comp
-L power:GND #PWR0109
-U 1 1 60ED62D7
-P 9350 5500
-F 0 "#PWR0109" H 9350 5250 50  0001 C CNN
-F 1 "GND" H 9350 5350 50  0000 C CNN
-F 2 "" H 9350 5500 50  0001 C CNN
-F 3 "" H 9350 5500 50  0001 C CNN
-	1    9350 5500
-	1    0    0    -1
-$EndComp
 Wire Wire Line
 	2450 4000 2550 4000
@@
 	2550 4300 2550 4400
 Connection ~ 2550 4400
-Text HLabel 10200 4950 2    50   Output ~ 0
-digital
-$Comp
-L Device:Jumper_NO_Small JP3
-U 1 1 60F1E267
-P 10000 4600
-F 0 "JP3" V 9954 4648 50  0000 L CNN
-F 1 "Jumper_NO_Small" V 10045 4648 50  0000 L CNN
-F 2 "Jumper:SolderJumper-2_P1.3mm_Open_Pad1.0x1.5mm" H 10000 4600 50  0001 C CNN
-F 3 "~" H 10000 4600 50  0001 C CNN
-	1    10000 4600
-	0    1    1    0
-$EndComp
-$Comp
-L Device:Jumper_NO_Small JP2
-U 1 1 60F1F64C
-P 9900 4950
-F 0 "JP2" H 9900 4765 50  0000 C CNN
-F 1 "Jumper_NO_Small" H 9900 4856 50  0000 C CNN
-F 2 "Jumper:SolderJumper-2_P1.3mm_Open_Pad1.0x1.5mm" H 9900 4950 50  0001 C CNN
-F 3 "~" H 9900 4950 50  0001 C CNN
-	1    9900 4950
-	-1   0    0    1
-$EndComp
-Wire Wire Line
-	10000 4950 10200 4950
-Wire Wire Line
-	10000 4700 10000 4950
-Connection ~ 10000 4950
 Wire Wire Line
 	10000 4500 10000 4000
@@
 	9250 4000 9900 4000
 Connection ~ 10000 4000
-Wire Wire Line
-	9250 4950 9800 4950
-Connection ~ 9250 4950
-$Comp
-L 0my_intf:MMCX J9
+$Comp
+L 0my_intf:MMCX J7
 U 1 1 6111E01B
 P 10100 3550
-F 0 "J9" H 10200 3525 50  0000 L CNN
+F 0 "J7" H 10200 3525 50  0000 L CNN
 F 1 "MMCX" H 10200 3434 50  0000 L CNN
 F 2 "0my_footprints:MMCX_JLC" H 10100 3550 50  0001 C CNN
@@
 	9900 4000 10000 4000
 $Comp
-L power:GND #PWR0114
+L power:GND #PWR020
 U 1 1 6112025C
 P 10100 3750
-F 0 "#PWR0114" H 10100 3500 50  0001 C CNN
+F 0 "#PWR020" H 10100 3500 50  0001 C CNN
 F 1 "GND" H 10100 3600 50  0000 C CNN
 F 2 "" H 10100 3750 50  0001 C CNN
@@
 $EndComp
 $Comp
-L power:PWR_FLAG #FLG0101
+L power:PWR_FLAG #FLG01
 U 1 1 612BA636
 P 3300 4000
-F 0 "#FLG0101" H 3300 4075 50  0001 C CNN
+F 0 "#FLG01" H 3300 4075 50  0001 C CNN
 F 1 "PWR_FLAG" H 3300 4173 50  0000 C CNN
 F 2 "" H 3300 4000 50  0001 C CNN
@@
 	3300 4000 3400 4000
 $Comp
-L power:PWR_FLAG #FLG0102
+L power:PWR_FLAG #FLG02
 U 1 1 612BABB0
 P 7950 4000
-F 0 "#FLG0102" H 7950 4075 50  0001 C CNN
+F 0 "#FLG02" H 7950 4075 50  0001 C CNN
 F 1 "PWR_FLAG" H 7950 4173 50  0000 C CNN
 F 2 "" H 7950 4000 50  0001 C CNN
@@
 Wire Wire Line
 	7950 4000 8150 4000
-$Comp
-L power:VCC #PWR0119
-U 1 1 62A18ABD
-P 2550 4000
-F 0 "#PWR0119" H 2550 3850 50  0001 C CNN
-F 1 "VCC" H 2567 4173 50  0000 C CNN
-F 2 "" H 2550 4000 50  0001 C CNN
-F 3 "" H 2550 4000 50  0001 C CNN
-	1    2550 4000
-	1    0    0    -1
-$EndComp
+Text HLabel 2450 4000 0    50   Input ~ 0
+power_in
+Text HLabel 2450 4400 0    50   Input ~ 0
+gnd_in
+Wire Wire Line
+	2450 4400 2550 4400
+Wire Wire Line
+	7700 4000 7950 4000
 $EndSCHEMATC
